File: pcb+power/kamstrup-wifi.sch (EAGLE design)
At the start: 22 parts, among them T1 BT137, T2 BT137

Commit message: pcb: v.1.1.4
better place for te terminal connectors
Parts:
- JP1, JP2, JP3: device SparkFun-Connectors:M025MM -> TE Terminal Block 45 degrees:M025MM
Changed lines of the file:
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@@
 <part name="R9" library="rcl" deviceset="R-EU_" device="R0805" value="39"/>
 <part name="C2" library="rcl" deviceset="C-EU" device="C1206" value="10nF"/>
-<part name="JP3" library="SparkFun-Connectors" deviceset="M02" device="5MM" value="AC OUT 2"/>
+<part name="JP3" library="TE Terminal Block 45 degrees" deviceset="M02" device="5MM" value="AC OUT 2"/>
 <part name="OK1" library="optocoupler" deviceset="MOC30*" device="S" technology="43" value="MOC3063S"/>
 <part name="GND2" library="SparkFun-Aesthetics" deviceset="GND" device=""/>
@@
 <part name="R5" library="rcl" deviceset="R-EU_" device="R0805" value="39"/>
 <part name="C1" library="rcl" deviceset="C-EU" device="C1206" value="10nF"/>
-<part name="JP1" library="SparkFun-Connectors" deviceset="M02" device="5MM" value="AC IN"/>
-<part name="JP2" library="SparkFun-Connectors" deviceset="M02" device="5MM" value="AC OUT 1"/>
+<part name="JP1" library="TE Terminal Block 45 degrees" deviceset="M02" device="5MM" value="AC IN"/>
+<part name="JP2" library="TE Terminal Block 45 degrees" deviceset="M02" device="5MM" value="AC OUT 1"/>
 <part name="T1" library="Triac SOT428" deviceset="BT137" device=""/>
 <part name="T2" library="Triac SOT428" deviceset="BT137" device=""/>
